File: hexar-flex/hexar-flex.kicad_sch (KiCad schematic)
At the start: 136 parts, among them J1 Conn_01x03, J10 6D, J11 +, J12 A9, J13 Photodiode, J14 -, J15 Conn_01x03_Socket, J17 8A, J18 RB W4, J19 7D, J2 B4, J20 7D, J21 NE W4, J22 9T, J23 9L, J3 DX, J4 Conn_01x02, J6 19 AD, J7 6D, J8 8D, J9 6D, Q1 8D, Q2 DX 18, Q3 6D, Q4 BK, SW1 SW_Push, SW2 SW_Push, SW3 SW_Push, SW4 SW_Push, U1 BR93CS46, U3 LB1837, U6 3.3V LDO, U7 IR3S64N1/T1, Y1 32768Hz?, Y2 2.00MHz

Commit message: WIP
Parts:
- C1: value 15.5n -> 15n; LCSC (none) -> C1644; Marking (none) -> 15.5n
- C10: value 108n -> 100n; LCSC (none) -> C14663; Marking (none) -> 108n
- C11, C12: value 115n -> 100n; LCSC (none) -> C14663; Marking (none) -> 115n
- C13, C14: LCSC (none) -> X; Manufacturer (none) -> Rubycon; Marking (none) -> 10u/10V; Part Number (none) -> TBD
- C15, C16: value 10p? -> 10p; LCSC (none) -> C1634; Marking (none) -> 10p?
- C17, C18: value 19p? -> 18p; LCSC (none) -> C1647; Marking (none) -> 19p?
- C2: value 334V 35uF -> 334V 35uF ESR??; Marking (none) -> 334V 35uF
- C3: LCSC (none) -> C1664; Marking (none) -> 330p
- C4: LCSC (none) -> C28233; Marking (none) -> 100n
- C5, C6: Manufacturer (none) -> Vishay; Marking (none) -> V684 680n ESR4R; Part Number (none) -> TR3A684K035C4000
- C7: value 34.5n -> 33n; LCSC (none) -> C1739; Marking (none) -> 34.5n
- C8: value 750n -> 1u; LCSC (none) -> C28323; Marking (none) -> 750n
- C9: value 34n -> 33n; LCSC (none) -> C1739; Marking (none) -> 34n
- D1: value D -> 5.6V?; symbol Device:D -> Device:D_Zener; LCSC (none) -> C282535; Manufacturer (none) -> Nexperia; Part Number (none) -> BZV55-B5V6,115
- D2, D3, D4: value 75W -> TVS?; LCSC (none) -> C111172; Manufacturer (none) -> onsemi; Marking (none) -> 75W; Part Number (none) -> SM05T1G
- D5: now left out of the parts list
- D7: renamed from J2; value B4 -> 1SS184; Manufacturer (none) -> Toshiba; Marking (none) -> B4; Part Number (none) -> 1SS184
- D8: renamed from J12; value A9 -> 1SS294; Manufacturer (none) -> Toshiba; Marking (none) -> A9; Part Number (none) -> 1SS294
- J3: Marking (none) -> DX
- Q1: value 8D -> UN2214; symbol Device:Q_NPN_BEC -> Device:Q_NPN_BEC_BRT; LCSC (none) -> C154618; Manufacturer (none) -> onsemi; Marking (none) -> 8D; Part Number (none) -> SMMUN2214LT1G
- Q10: renamed from J20; value 7D -> UN2124; symbol Device:Q_PNP_BEC -> Device:Q_PNP_BEC_BRT; Marking (none) -> 7D
- Q11: renamed from J9; value 6D -> UN2114; symbol Device:Q_PNP_BEC -> Device:Q_PNP_BEC_BRT; LCSC (none) -> C232565; Manufacturer (none) -> onsemi; Marking (none) -> 6D; Part Number (none) -> MUN2114T1G
- Q12: renamed from J8; value 8D -> UN2214; symbol Device:Q_NPN_BEC -> Device:Q_NPN_BEC_BRT; LCSC (none) -> C154618; Manufacturer (none) -> onsemi; Marking (none) -> 8D; Part Number (none) -> SMMUN2214LT1G
- Q13: renamed from J22; value 9T -> XN1211; Manufacturer (none) -> Panasonic; Marking (none) -> 9T; Part Number (none) -> XN1211
- Q14: renamed from J23; value 9L -> XN1213; Manufacturer (none) -> Panasonic; Marking (none) -> 9L; Part Number (none) -> XN1213
- Q2: value DX 18 -> HQ1A4A; symbol Connector_Generic:Conn_01x03 -> Device:Q_PNP_BCE; Manufacturer (none) -> NEC; Marking (none) -> DX 18; Part Number (none) -> HQ1A4A
- Q3: value 6D -> UN2114; symbol Device:Q_PNP_BEC -> Device:Q_PNP_BEC_BRT; LCSC (none) -> C232565; Manufacturer (none) -> onsemi; Marking (none) -> 6D; Part Number (none) -> MUN2114T1G
- Q4: Marking (none) -> BK
- Q5: renamed from J7; value 6D -> UN2114; symbol Device:Q_PNP_BEC -> Device:Q_PNP_BEC_BRT; LCSC (none) -> C232565; Manufacturer (none) -> onsemi; Marking (none) -> 6D; Part Number (none) -> MUN2114T1G
- Q6: renamed from J10; value 6D -> UN2114; symbol Device:Q_PNP_BEC -> Device:Q_PNP_BEC_BRT; LCSC (none) -> C232565; Manufacturer (none) -> onsemi; Marking (none) -> 6D; Part Number (none) -> MUN2114T1G
- Q7: renamed from J6; value 19 AD -> CR08AS-8; symbol Device:Q_NMOS_GDS -> Device:Q_SCR_GAK; LCSC (none) -> C151231; Manufacturer (none) -> Renesas; Marking (none) -> 19 AD; Part Number (none) -> CR08AS-12A
- Q8: renamed from J17; value 8A -> UN2211; symbol Device:Q_NPN_BEC -> Device:Q_NPN_BEC_BRT; LCSC (none) -> C232615; Manufacturer (none) -> onsemi; Marking (none) -> 8A; Part Number (none) -> MUN2211T1G
- Q9: renamed from J19; value 7D -> UN2124; symbol Device:Q_PNP_BEC -> Device:Q_PNP_BEC_BRT; Marking (none) -> 7D
- R1, R2, R3, R4, R5, R53, R6: value 514 -> 510k/1%; LCSC (none) -> C23192; Marking (none) -> 514
- R10: value 513 -> 51k/1%; LCSC (none) -> C23196; Marking (none) -> 513
- R11, R13, R14, R15, R16, R18, R19, R32, R35, R42, R47: value 104 -> 100k/1%; LCSC (none) -> C25803; Marking (none) -> 104
- R12: value 120 -> 12R/1%; LCSC (none) -> C25803; Marking (none) -> 120
- R17: value NTC 47k? -> NTC 50k?; LCSC (none) -> C338754; Marking (none) -> none
- R20, R21, R22, R23, R31, R37: value 204 -> 200k/1%; LCSC (none) -> C25811; Marking (none) -> 204
- R24, R52: value 102 -> 1k/1%; LCSC (none) -> C21190; Marking (none) -> 102
- R25, R26, R33: value 221 -> 220R/1%; LCSC (none) -> C22962; Marking (none) -> 221
- R27: value 511 -> 510R/1%; LCSC (none) -> C23193; Marking (none) -> 511
- R28: value 1R5 -> 1R5/1%; LCSC (none) -> C17392; Marking (none) -> 1R5
- R29: value 2R0 -> 2R0/1%; LCSC (none) -> C17606; Marking (none) -> 2R0
- R30: value 133 -> 13k/1%; LCSC (none) -> C22797; Marking (none) -> 133
- R34: value 391 -> 390R/1%; LCSC (none) -> C23151; Marking (none) -> 391
- R36: value 201 -> 200R/1%; LCSC (none) -> C8218; Marking (none) -> 201
- R38: value 563 -> 56k/1%; LCSC (none) -> C23206; Marking (none) -> 563
- R39: value 392 -> 3.9k/1%; LCSC (none) -> C23018; Marking (none) -> 392
- R40, R43: value 562 -> 5.6k/1%; LCSC (none) -> C23189; Marking (none) -> 562
- R41, R44: value 162 -> 1.6k/1%; LCSC (none) -> C22847; Marking (none) -> 162
- R45: value 362 -> 3.6k/1%; LCSC (none) -> C22980; Marking (none) -> 362
- R46: value 512 -> 5.1k/1%; LCSC (none) -> C23186; Marking (none) -> 512
- R48: value 153 -> 15k/1%; LCSC (none) -> C22809; Marking (none) -> 153
- R49: value 106 -> 10M/1%; LCSC (none) -> C7250; Marking (none) -> 106
- R50, R9: value 105 -> 1M/1%; LCSC (none) -> C22935; Marking (none) -> 105
- R51: value 334 -> 330k/1%; LCSC (none) -> C23137; Marking (none) -> 334
- R54: value 243 -> 24k/1%; LCSC (none) -> C23352; Marking (none) -> 243
- R55: value 163 -> 16k/1%; LCSC (none) -> C22818; Marking (none) -> 163
- R7: value 303 -> 30k/1%; LCSC (none) -> C22984; Marking (none) -> 303
- R8: value 203 -> 20k/1%; LCSC (none) -> C4184; Marking (none) -> 203
- U1: LCSC (none) -> X; Marking (none) -> CS46
- U10: renamed from J13; Manufacturer (none) -> Sharp; Marking (none) -> S 3040 18 G9
- U2: value ~ -> M37423M8H-101FP; LCSC (none) -> X; Manufacturer (none) -> Mitsubishi; Part Number (none) -> M37423M8H-101FP
- U3: value LB1837 -> LB1837M; LCSC (none) -> X; Marking (none) -> LB1837
- U4, U5: value ~ -> LB8620M; LCSC (none) -> X; Marking (none) -> LB8620
- U6: value 3.3V LDO -> 3.3V? LDO; LCSC (none) -> C27287; Manufacturer (none) -> Microchip; Marking (none) -> OK 09; Part Number (none) -> MCP1703T-3302E/MB
- U7: LCSC (none) -> X; Marking (none) -> 3S64
- U8: renamed from J21; value NE W4 -> S-8052ANB-NE?; symbol Connector_Generic:Conn_01x03 -> Power_Supervisor:MCP100-300D; Manufacturer (none) -> Epson; Marking (none) -> NE W4; Part Number (none) -> S-8052ANB-NE
- U9: renamed from J18; value RB W4 -> S-81230AG?; symbol Connector_Generic:Conn_01x03 -> Regulator_Linear:MCP1703Ax-330xxMB; Manufacturer (none) -> Seiko; Marking (none) -> RB W4; Part Number (none) -> S-81230AG
Connections:
- net VDRV3 is gone; now on net +BATT: D8.1 (Pin_1), Q11.2 (E), Q5.2 (E), Q6.2 (E), R34.1, U3.14 (VCC)
- net GND: now also R54.2; no longer J1.2 (Pin_2)
- net P58: now also Q14.5 (Pin_5)
- net P59: now also Q14.4 (Pin_4)
- net VXXX: now also C12.1, R47.2, U9.3 (VO)
- net at R36.1: now also J1.2 (Pin_2)
- net P37 renamed P37/RESET
Other:
- note added: "3V LDO?"
- note added: "E-B 10k"
- note added: "Power supervisor"
- note added: "Reset?"
- moved on the sheet: C11, C12, D5, D6, D8, Q13, R28, R29, R34, R36, R46, R47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

Commit message: WIP
Parts:
- added DS1: HEXAR-LCD, flex-smd:HEXAR-LCD, symbol Connector_Generic_Shielded:Conn_02x10_Counter_Clockwise_Shielded
- added J2: Conn_01x10, symbol Connector_Generic:Conn_01x10
- C13, C14: Part Number TBD -> 10ML100MEFC6.3X5
- D7: LCSC (none) -> C165922; Marking B4 -> B3
- D8: symbol Connector_Generic:Conn_01x03 -> Library:1SS294; LCSC (none) -> C261914
Connections:
- net GND: now also SW4.2, DS1.SH (Shield), J2.2 (Pin_2), J2.8 (Pin_8)
- net P100: now also J2.9 (Pin_9)
- net P35: now also J2.1 (Pin_1)
- net P44: now also J2.5 (Pin_5)
- net P63: now also J2.4 (Pin_4)
- net P67: now also J2.6 (Pin_6)
- net P68: now also J2.7 (Pin_7)
- net P74: now also J2.3 (Pin_3)
- net P78: now also DS1.12 (Pin_12)
- net P79: now also DS1.14 (Pin_14)
- net P82: now also DS1.10 (Pin_10)
- net P83: now also DS1.9 (Pin_9)
- net P84: now also DS1.8 (Pin_8)
- net P85: now also DS1.7 (Pin_7)
- net P86: now also DS1.6 (Pin_6)
- net P87: now also DS1.5 (Pin_5)
- net P88: now also DS1.4 (Pin_4)
- net P89: now also DS1.13 (Pin_13)
- net P90: now also DS1.16 (Pin_16)
- net P91: now also DS1.3 (Pin_3)
- net P92: now also DS1.19 (Pin_19)
- net P93: now also DS1.18 (Pin_18), DS1.2 (Pin_2)
- net P94: now also DS1.17 (Pin_17)
- net P95: now also DS1.15 (Pin_15)
- net VDD: now also J2.10 (Pin_10)
- no-connect marks 0 -> 3
Other:
- moved on the sheet: C10, C11, C12, C13, C14, J11, J14, Q4A, Q4B, R46, R47, SW1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

Commit message: WIP
Parts:
- added J10, J8: -, TestPoint:TestPoint_Pad_D1.5mm, symbol Connector:Conn_01x01_Socket
- added J12: OUT, TestPoint:TestPoint_Pad_D1.5mm, symbol Connector:Conn_01x01_Socket
- added J13: IN, TestPoint:TestPoint_Pad_D1.5mm, symbol Connector:Conn_01x01_Socket
- added J16: GND, TestPoint:TestPoint_Pad_D1.5mm, symbol Connector:Conn_01x01_Socket
- added J5: Conn_01x12_MountingPin, flex-smd:FFC-12, symbol Connector_Generic_MountingPin:Conn_01x12_MountingPin
- added J6: Conn_01x08_MountingPin, flex-smd:FFC-8, symbol Connector_Generic_MountingPin:Conn_01x08_MountingPin
- added J7, J9: +, TestPoint:TestPoint_Pad_D1.5mm, symbol Connector:Conn_01x01_Socket
- added TP19: 3VSW, flex-smd:TestPoint_Pad_D1.2mm, symbol Connector:TestPoint
- added TP20: 3VALW, flex-smd:TestPoint_Pad_D1.2mm, symbol Connector:TestPoint
- added TP21: BATTSW, flex-smd:TestPoint_Pad_D1.2mm, symbol Connector:TestPoint
- added TP22: RESET, flex-smd:TestPoint_Pad_D1.2mm, symbol Connector:TestPoint
- added TP23: P42SW, flex-smd:TestPoint_Pad_D1.2mm, symbol Connector:TestPoint
- added TP24: P58, flex-smd:TestPoint_Pad_D1.2mm, symbol Connector:TestPoint
- added TP25: P59, flex-smd:TestPoint_Pad_D1.2mm, symbol Connector:TestPoint
- added TP26: P24, flex-smd:TestPoint_Pad_D1.2mm, symbol Connector:TestPoint
- added TP27, TP65: P25, flex-smd:TestPoint_Pad_D1.2mm, symbol Connector:TestPoint
- added TP28: P69, flex-smd:TestPoint_Pad_D1.2mm, symbol Connector:TestPoint
- added TP29: P59IN, flex-smd:TestPoint_Pad_D1.2mm, symbol Connector:TestPoint
- added TP30: M1+, flex-smd:TestPoint_Pad_D1.2mm, symbol Connector:TestPoint
- added TP31: M1-, flex-smd:TestPoint_Pad_D1.2mm, symbol Connector:TestPoint
- added TP33: P57, flex-smd:TestPoint_Pad_D1.2mm, symbol Connector:TestPoint
- added TP34: P46SW, flex-smd:TestPoint_Pad_D1.2mm, symbol Connector:TestPoint
- added TP35: P47SW, flex-smd:TestPoint_Pad_D1.2mm, symbol Connector:TestPoint
- added TP36: P48SW, flex-smd:TestPoint_Pad_D1.2mm, symbol Connector:TestPoint
- added TP37, TP40: GND, flex-smd:TestPoint_Pad_D1.2mm, symbol Connector:TestPoint
- added TP38: P3, flex-smd:TestPoint_Pad_D1.2mm, symbol Connector:TestPoint
- added TP39: BATT, flex-smd:TestPoint_Pad_D1.2mm, symbol Connector:TestPoint
- added TP41: CAP2, flex-smd:TestPoint_Pad_D1.2mm, symbol Connector:TestPoint
- added TP42: M2+, flex-smd:TestPoint_Pad_D1.2mm, symbol Connector:TestPoint
- added TP43: M2-, flex-smd:TestPoint_Pad_D1.2mm, symbol Connector:TestPoint
- added TP44: M5+, flex-smd:TestPoint_Pad_D1.2mm, symbol Connector:TestPoint
- added TP45: M5-, flex-smd:TestPoint_Pad_D1.2mm, symbol Connector:TestPoint
- added TP46: M6-, flex-smd:TestPoint_Pad_D1.2mm, symbol Connector:TestPoint
- added TP47: M6+, flex-smd:TestPoint_Pad_D1.2mm, symbol Connector:TestPoint
- added TP48: M4+, flex-smd:TestPoint_Pad_D1.2mm, symbol Connector:TestPoint
- added TP49: M4-, flex-smd:TestPoint_Pad_D1.2mm, symbol Connector:TestPoint
- added TP50: SELF, flex-smd:TestPoint_Pad_D1.2mm, symbol Connector:TestPoint
- added TP51: P70, flex-smd:TestPoint_Pad_D1.2mm, symbol Connector:TestPoint
- added TP52: IRK, flex-smd:TestPoint_Pad_D1.2mm, symbol Connector:TestPoint
- added TP53: FLASH, flex-smd:TestPoint_Pad_D1.2mm, symbol Connector:TestPoint
- added TP54: IRA, flex-smd:TestPoint_Pad_D1.2mm, symbol Connector:TestPoint
- added TP55: R, flex-smd:TestPoint_Pad_D1.2mm, symbol Connector:TestPoint
- added TP56: MF, flex-smd:TestPoint_Pad_D1.2mm, symbol Connector:TestPoint
- added TP57: SEL, flex-smd:TestPoint_Pad_D1.2mm, symbol Connector:TestPoint
- added TP58: FLD, flex-smd:TestPoint_Pad_D1.2mm, symbol Connector:TestPoint
- added TP59: A, flex-smd:TestPoint_Pad_D1.2mm, symbol Connector:TestPoint
- added TP60: PSD1, flex-smd:TestPoint_Pad_D1.2mm, symbol Connector:TestPoint
- added TP61: PSD2, flex-smd:TestPoint_Pad_D1.2mm, symbol Connector:TestPoint
- added TP62: VPSD, flex-smd:TestPoint_Pad_D1.2mm, symbol Connector:TestPoint
- added TP63: P71, flex-smd:TestPoint_Pad_D1.2mm, symbol Connector:TestPoint
- added TP64: P72, flex-smd:TestPoint_Pad_D1.2mm, symbol Connector:TestPoint
- added TP66: P69SW, flex-smd:TestPoint_Pad_D1.2mm, symbol Connector:TestPoint
- added TP67: P25SW, flex-smd:TestPoint_Pad_D1.2mm, symbol Connector:TestPoint
- added TP69: P24IN, flex-smd:TestPoint_Pad_D1.2mm, symbol Connector:TestPoint
- added TP71: P58IN, flex-smd:TestPoint_Pad_D1.2mm, symbol Connector:TestPoint
- C2: value 334V 35uF ESR?? -> 33u/35V
- C5, C6: value V684 680n ESR4R -> 0.68u/35V
- D1: value 5.6V? -> 7.5V; LCSC C282535 -> C426817; Part Number BZV55-B5V6,115 -> BZV55-C7V5,115
- D7: symbol Connector_Generic:Conn_01x03 -> Device:D_Dual_CommonCathode_AKA
- J1: value Conn_01x03 -> ???; footprint (none) -> flex-smd:CUSTOM-3
- Q4: symbol Device:Q_Dual_PMOS_S1G1D2S2G2D1 -> Device:Q_Dual_PNP_PNP_E1B1C2E2B2C1
- R17: value NTC 50k? -> NTC 64k@25C B=4000; LCSC C338754 -> (none)
- TP1, TP10, TP16, TP17, TP2, TP3, TP4, TP5, TP6: footprint flex-smd:TestPoint_Pad_D1.8mm_A1.2mm -> flex-smd:TestPoint_Pad_D1.2mm
- TP11: value P11 -> DO; footprint flex-smd:TestPoint_Pad_D1.8mm_A1.2mm -> flex-smd:TestPoint_Pad_D1.2mm
- TP12: value P12 -> DI; footprint flex-smd:TestPoint_Pad_D1.8mm_A1.2mm -> flex-smd:TestPoint_Pad_D1.2mm
- TP13: value P13 -> SK; footprint flex-smd:TestPoint_Pad_D1.8mm_A1.2mm -> flex-smd:TestPoint_Pad_D1.2mm
- TP14: value P14 -> CS; footprint flex-smd:TestPoint_Pad_D1.8mm_A1.2mm -> flex-smd:TestPoint_Pad_D1.2mm
- TP15: value P21 -> IR2; footprint flex-smd:TestPoint_Pad_D1.8mm_A1.2mm -> flex-smd:TestPoint_Pad_D1.2mm
- TP18: value 3.3V -> 3V_AUX; footprint flex-smd:TestPoint_Pad_D1.8mm_A1.2mm -> flex-smd:TestPoint_Pad_D1.2mm
- TP7: value P1 -> NTC; footprint flex-smd:TestPoint_Pad_D1.8mm_A1.2mm -> flex-smd:TestPoint_Pad_D1.2mm
- TP8: value P2 -> VBAT; footprint flex-smd:TestPoint_Pad_D1.8mm_A1.2mm -> flex-smd:TestPoint_Pad_D1.2mm
- TP9: value P9 -> IR1; footprint flex-smd:TestPoint_Pad_D1.8mm_A1.2mm -> flex-smd:TestPoint_Pad_D1.2mm
- U6: value 3.3V? LDO -> LDO 3.0V Iq=1.3uA; Part Number MCP1703T-3302E/MB -> MCP1703T-3002E/MB
- U9: value S-81230AG? -> LDO 3.0V Iq=1.3uA
Connections:
- net VXXX is gone; now on net +3V_ALW: C12.1, Q4.4 (E2), R1.1, R12.1, R2.1, R3.1, R4.1, R47.2, R5.1, R53.1, R6.2, U2.8, U9.3 (VO)
- net Vc2 is gone; now on net Vc12: U3.5 (Vc2)
- net +BATT: now also TP39.1
- net +BATTSW: now also TP21.1
- net CAP2: now also TP41.1
- net FLASH_IN: now also J13.1 (Pin_1)
- net FLASH_OUT: now also J12.1 (Pin_1)
- net GND: now also J10.1 (Pin_1), J16.1 (Pin_1), J5.2 (Pin_2), J6.4 (Pin_4), TP37.1, TP40.1
- net IR_A: now also TP54.1
- net IR_SNS: now also TP52.1
- net M1+: now also J6.7 (Pin_7), TP30.1
- net M1-: now also J6.8 (Pin_8), TP31.1
- net M2+: now also J5.5 (Pin_5), TP42.1
- net M2-: now also J5.6 (Pin_6), TP43.1
- net M3+: now also J7.1 (Pin_1)
- net M3-: now also J8.1 (Pin_1)
- net M4+: now also J5.7 (Pin_7), TP48.1
- net M4-: now also J5.8 (Pin_8), TP49.1
- net M5+: now also J5.9 (Pin_9), TP44.1
- net M5-: now also J5.10 (Pin_10), TP45.1
- net M6+: now also J5.11 (Pin_11), TP47.1
- net M6-: now also J5.12 (Pin_12), TP46.1
- net P24: now also TP26.1
- net P24IN: now also J6.5 (Pin_5), TP69.1
- net P25: now also TP27.1
- net P26: now also TP65.1
- net P32: no longer R1.2
- net P37/RESET: now also TP22.1
- net P41SW: now also J5.3 (Pin_3)
- net P42SW: now also J6.1 (Pin_1), J6.6 (Pin_6), TP23.1
- net P44: no longer J2.5 (Pin_5), R6.1, TP17.1, U2.44
- net P46SW: now also TP34.1
- net P47SW: now also TP35.1
- net P48SW: now also TP36.1
- net P57: now also TP33.1
- net P58: now also TP24.1
- net P59: now also TP25.1
- net P69: now also TP28.1
- net P70: now also TP51.1
- net P71: now also TP63.1
- net P72: now also TP64.1
- net PSD1: now also TP60.1
- net PSD2: now also TP61.1
- net VPSD: now also TP62.1
- net P59IN: now reaches R54.1
- net P59IN: now also Q14.3 (Pin_3), J5.1 (Pin_1), TP29.1
- net P69SW: now reaches Q13.1 (Pin_1)
- net P69SW: now also J6.2 (Pin_2), TP66.1
- net P25SW: now reaches Q13.3 (Pin_3)
- net P25SW: now also J6.3 (Pin_3), TP67.1
- net P58IN: now reaches Q14.1 (Pin_1), R55.1
- net P58IN: now also J5.4 (Pin_4), TP71.1
- net +3.3V renamed +3V_AUX
- net P10 renamed P10/UNUSED
- net P100 renamed P100/A_ADC
- net P100/A_ADC: now also TP59.1
- net P19 renamed P19/CONT34
- net P20 renamed P20/CONT12
- net P21 renamed P21/IR2
- net P22 renamed P22/FLASH
- net P22/FLASH: now also TP53.1
- net P23 renamed P23/PULLUP
- net P3 renamed P3/CUTOFF
- net P3/CUTOFF: now also TP38.1
- net P31 renamed P31/3VSW
- net P35 renamed P35/SW?
- net P43 renamed P43/BATTSW
- net P45 renamed P45/SELFLED
- net P49 renamed P49/M2INB
- net P50 renamed P50/M2INA
- net P51 renamed P51/M12IND
- net P52 renamed P52/M12INC
- net P53 renamed P53/M1INB
- net P54 renamed P54/M1INA
- net P61 renamed P61/SW_DOOR
- net P61/SW_DOOR: now also J9.1 (Pin_1)
- net P62 renamed P62/SW_R
- net P62/SW_R: now also TP55.1
- net P63 renamed P63/SW?
- net P64 renamed P64/SW_SELF
- net P64/SW_SELF: now also TP50.1
- net P65 renamed P65/SW_MF
- net P65/SW_MF: now also TP56.1
- net P66 renamed P66/SW_SELECT
- net P66/SW_SELECT: now also TP57.1
- net P67 renamed P67/SW?
- net P68 renamed P68/SW?
- net P73 renamed P73/FLASH_DATA
- net P73/FLASH_DATA: now also TP58.1
- net P74 renamed P74/SW?
- net P75 renamed +3V_ALW
- net +3V_ALW: now also TP20.1
- net P77: no longer names the net of U2.77
- net P78 renamed P78/LCD
- net P79 renamed P79/LCD
- net P80: no longer names the net of U2.80
- net P81: no longer names the net of U2.81
- net P82 renamed P82/LCD
- net P83 renamed P83/LCD
- net P84 renamed P84/LCD
- net P85 renamed P85/LCD
- net P86 renamed P86/LCD
- net P87 renamed P87/LCD
- net P88 renamed P88/LCD
- net P89 renamed P89/LCD
- net P9 renamed P9/IR1
- net P90 renamed P90/LCD
- net P91 renamed P91/LCD
- net P92 renamed P92/LCD
- net P93 renamed P93/LCD
- net P94 renamed P94/LCD
- net P95 renamed P95/LCD
- net P96: no longer names the net of U2.96
- net P97: no longer names the net of U2.97
- net P98: no longer names the net of U2.98
- net P99: no longer names the net of U2.99
- net VDD renamed +3V_SW
- net +3V_SW: now also TP19.1
- net Vc1 renamed Vc12
- new net P32/SW?: R1.2
- new net P44/SW?: J2.5 (Pin_5), TP17.1, U2.44
- new net P44//SW?: R6.1
- no-connect marks 3 -> 10
Other:
- note added: "3.0V rail for CPU active, DX code reader, NTC, EEPROM, etc."
- note added: "3.0V rail for CPU standby and always-on things like keyboard, also regulated 3.0V to photodiode"
- note added: "???"
- note added: "Both LDO: 3.0V Iq=1.3uA"
- note added: "DX READER"
- note added: "EEPROM"
- note added: "EXPOSURE SENSOR"
- note added: "FLASH"
- note added: "KEYBOARD"
- note added: "LCD"
- note added: "MCU"
- note added: "MISC"
- note added: "MOTOR DRIVERS"
- note added: "Matching: LBC848BPDW1T3G"
- note added: "PSD/AUTOFOCUS"
- note added: "Possibly 3.0V rail for high load peripherals"
- note added: "SHARP IR3S64 see: SHARP IR3S71 https://www.digchip.com/datasheets/parts/datasheet/2308/IR3S85-pdf.php"
- note added: "SUPPLY"
- note added: "Switched battery rail for voltage measurement and photodiode"
- note added: "TODO: This diode is problematic, high Vf at moderate currents. Measure the same diode from the second camera perhaps?"
- note added: "TVS are originally 7.5V zeners :)"
- note added: "To FFC"
- note removed: "3V LDO?"
- note removed: "Power supervisor"
- note removed: "Reset?"
- note removed: "SHARP IR3S64 see: SHARP IR3S71 https://www.digchip.com/datasheets/parts/datasheet/2308/IR3S85-pdf.php IR3S64N1/T1 SSOP-12"
- note removed: "TODO: Verify"
- moved on the sheet: C1, C10, C11, C12, C13, C14, C15, C16, C17, C18, C2, C3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

Commit message: WIP
Parts:
- removed TP1: SD, flex-smd:TestPoint_Pad_D1.2mm, symbol Connector:TestPoint
- removed TP3: S2, flex-smd:TestPoint_Pad_D1.2mm, symbol Connector:TestPoint
- added D101, D102: SHARP-PSD, flex-smd:SHARP-PSD, symbol Library:SHARP-PSD
- added J101: Conn_01x04, flex-smd:HEXAR-SOLD4PIN, symbol Connector_Generic:Conn_01x04
- added SW101: SKRNPME010, flex-smd:ALPS-SKRN, symbol Library:SKRNPME010
- added TP101: P60, flex-smd:TestPoint_Pad_D1.2mm, symbol Connector:TestPoint
- added TP102: P32, flex-smd:TestPoint_Pad_D1.2mm, symbol Connector:TestPoint
- added TP103: P68, flex-smd:TestPoint_Pad_D1.2mm, symbol Connector:TestPoint
- added TP104: GND, flex-smd:TestPoint_Pad_D1.2mm, symbol Connector:TestPoint
- added TP105: SL, flex-smd:TestPoint_Pad_D1.2mm, symbol Connector:TestPoint
- J3: footprint (none) -> flex-smd:HEXAR-DX
- R1, R10, R11, R12, R13, R14, R15, R16, R18, R19, R2, R20, R21, R22, R23, R24, R25, R26, R27, R3, R30, R31, R32, R33, R34, R35, R36, R37, R38, R39, R4, R40, R41, R42, R43, R44, R45, R46, R47, R48, R5, R50, R51, R52, R53, R54, R55, R6, R7, R8, R9: footprint Resistor_SMD:R_0603_1608Metric -> flex-smd:R_0603_SMD
Connections:
- net GND: now also D101.4 (GND), D102.4 (GND), J101.4 (Pin_4), SW101.2, SW101.3, SW101.5, SW101.6, TP104.1
- net P32: now also TP102.1
- net P46SW: now also J101.1 (Pin_1)
- net P47SW: now also J101.3 (Pin_3)
- net P48SW: now also J101.2 (Pin_2)
- net P60: now also TP101.1
- net P68/SW?: now also TP103.1
- net PSD1: now also D101.2 (K1), D102.2 (K1)
- net PSD2: now also D101.3 (K2), D102.3 (K2)
- net SELFLEDA: now also TP105.1
- net VPSD: now also D101.1 (A), D102.1 (A)
Other:
- moved on the sheet: Q11, Q5, Q6, R25, R26, R33, TP34, TP35, TP36, TP37

Commit message: hexar-flex: WIP
Parts:
- removed J15: Conn_01x03_Socket, symbol Connector:Conn_01x03_Socket
- added Q15: Q_Dual_NPN_C2C1E1E2, symbol Device:Q_Dual_NPN_C2C1E1E2
- C13, C14: value 10u/10V -> 100u/10V
- U9: LCSC (none) -> C27287
Other:
- note added: "ANALOG INPUTS"
- note added: "DOOR SENSOR"
- note added: "LED"
- note added: "M3: Positive = rewind M3: Negative = wind"
- note added: "OUTPUT DRIVERS TODO: Label signals"
- note added: "SHUTTER RELEASE"
- note added: "TODO: List NO/NC"
- note added: "TODO: Proper symbols for these transistors"
- note added: "TODO: Replace with original footprint"
- note added: "UNKNOWN INPUT"
- note added: "UNKNOWN SENSOR"
- note added: "UNKNOWN SERVICE INPUT"
- note removed: "MISC"
- moved on the sheet: C1, C10, C11, C12, C13, C14, C15, C16, C17, C18, C2, C3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
